File: stm32f042cXt6_demo/stm32f042cXt6_demo.kicad_pcb (KiCad board)
At the start: 2 copper layers, 75 x 75 mm, 64 parts, among them J1 PGM, J2 USB_B_Micro, J3 EXT, M1 AM4311T42A0, P1 S2, P10 PB4, P11 S0, P12 PB5, P13 S3, P14 PB6, P15 S1, P16 PB7, P17 S5, P18 PB8, P19 S4, P2 PB0, P20 PB9, P21 S3, P22 PB10, P23 TA10, P24 S2, P25 PB11, P26 S1, P27 PB12, P28 S0, P29 PB13, P3 S0, P30 PB14, P31 PB15, P32 TA8, P33 TA9, P34 CONN_1, P35 CONN_1, P36 CONN_1, P37 CONN_1, P4 PB1, P5 S5, P6 PB2, P7 S2, P8 PB3, P9 S4, SW1 TACTILE, U1 STM32F042C4Tx, U2 AZ1117-3.3, U3 USB_PROTECTION, U4 LTR-553ALS-WA

Commit message: Bump
Other:
- rule pad_to_mask_clearance: 0.051 -> 0.02
- rule solder_mask_min_width: 0.25 -> 0.3
Changed lines of the file:
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@@
-(kicad_pcb (version 20171130) (host pcbnew "(5.1.4)-1")
+(kicad_pcb (version 20171130) (host pcbnew 5.1.5-52549c5~84~ubuntu18.04.1)
   (general
     (thickness 1.6)
@@
     (pad_size 0.4826 0.4826)
     (pad_drill 0)
-    (pad_to_mask_clearance 0.051)
-    (solder_mask_min_width 0.25)
+    (pad_to_mask_clearance 0.02)
+    (solder_mask_min_width 0.3)
     (aux_axis_origin 0 0)
     (visible_elements 7FFFFFFF)
