File: stm32f042cXt6_demo/stm32f042cXt6_demo.sch (KiCad schematic (older format))
At the start: 64 parts, among them J1 PGM, J2 USB_B_Micro, J3 EXT, M1 AM4311T42A0, P1 S2, P10 PB4, P11 S0, P12 PB5, P13 S3, P14 PB6, P15 S1, P16 PB7, P17 S5, P18 PB8, P19 S4, P2 PB0, P20 PB9, P21 S3, P22 PB10, P23 TA10, P24 S2, P25 PB11, P26 S1, P27 PB12, P28 S0, P29 PB13, P3 S0, P30 PB14, P31 PB15, P32 TA8, P33 TA9, P34 CONN_1, P35 CONN_1, P36 CONN_1, P37 CONN_1, P4 PB1, P5 S5, P6 PB2, P7 S2, P8 PB3, P9 S4, SW1 TACTILE, U1 STM32F042C4Tx, U2 AMS1117-3.3, U3 USB_PROTECTION, U4 LTR-553ALS-WA

Commit message: Bump
Parts:
- C1, C2, C3, C4, C5, C6: symbol 5050RGB:C -> stm32f042cXt6_demo-rescue:C-5050RGB
- D1, D2, D3, D4, D5, D6: symbol LED:WS2812B -> stm32f042cXt6_demo-rescue:WS2812B-LED
- J1: symbol Connector:Conn_01x05_Male -> stm32f042cXt6_demo-rescue:Conn_01x05_Male-Connector
- J2: symbol Connector:USB_B_Micro -> stm32f042cXt6_demo-rescue:USB_B_Micro-Connector
- J3: symbol Connector_Generic:Conn_02x03_Odd_Even -> stm32f042cXt6_demo-rescue:Conn_02x03_Odd_Even-Connector_Generic
- M1: symbol Connector_Generic:Conn_01x04 -> stm32f042cXt6_demo-rescue:Conn_01x04-Connector_Generic
- P1, P10, P11, P12, P13, P14, P15, P16, P17, P18, P19, P2, P20, P21, P22, P23, P24, P25, P26, P27, P28, P29, P3, P30, P31, P32, P33, P34, P35, P36, P37, P4, P5, P6, P7, P8, P9: symbol 5050RGB:CONN_1 -> stm32f042cXt6_demo-rescue:CONN_1-5050RGB
- R1, R2, R3, R4, R5, R6: symbol 5050RGB:R -> stm32f042cXt6_demo-rescue:R-5050RGB
- SW1: symbol tactile:TACTILE -> stm32f042cXt6_demo-rescue:TACTILE-tactile
- U1: symbol MCU_ST_STM32F0:STM32F042C4Tx -> stm32f042cXt6_demo-rescue:STM32F042C4Tx-MCU_ST_STM32F0
- U2: symbol Regulator_Linear:AZ1117-3.3 -> stm32f042cXt6_demo-rescue:AZ1117-3.3-Regulator_Linear
- U3: symbol usb-prot-ip4220cz6:USB-PROT-IP4220CZ6 -> stm32f042cXt6_demo-rescue:USB-PROT-IP4220CZ6-usb-prot-ip4220cz6
- U4: symbol kicad:LTR-553ALS-WA-LITE-ON-AMBIENT -> stm32f042cXt6_demo-rescue:LTR-553ALS-WA-LITE-ON-AMBIENT-kicad
