File: multitool/zeta_sim/sepic_sim.sch (KiCad schematic (older format))
At the start: 13 parts, among them Q1 Q_NMOS_DGS, Q2 Q_NMOS_DGS

Commit message: update some tweaks to the zeta sim thoughts.
Parts:
- Rload1: renamed from Rload; Spice_Model 20 -> 400
- Vpulse1: renamed from Vpulse?; Spice_Model dc 10 pulse(0 10 0u 100n 100n 2.5u 4.5u) -> dc 10 pulse(0 10 0u 100n 100n 1000n 3.5u)
- Vpulse2: renamed from Vpulse; Spice_Model dc 10 pulse(0 10 2.7u 100n 100n 1.2u 4.5u) -> dc 10 pulse(0 0 900n 100n 100n 700n 2.1u)
- gave numbers to parts that had none: 2
- renumbered Cmid to Cmid1, Cout to Cout1, Drect to Drect1, Lin to Lin1, Lout to Lout1, Rsource to Rsource1
Changed lines of the file:
@@
 $EndDescr
 $Comp
-L pspice:0 #GND?
+L pspice:0 #GND0101
 U 1 1 5EC9CCCB
 P 4350 4400
-F 0 "#GND?" H 4350 4300 50  0001 C CNN
+F 0 "#GND0101" H 4350 4300 50  0001 C CNN
 F 1 "0" H 4350 4489 50  0000 C CNN
 F 2 "" H 4350 4400 50  0001 C CNN
@@
 $EndComp
 $Comp
-L pspice:VSOURCE V?
+L pspice:VSOURCE V1
 U 1 1 5EC9E6CC
 P 1100 2750
-F 0 "V?" H 1328 2796 50  0000 L CNN
+F 0 "V1" H 1328 2796 50  0000 L CNN
 F 1 "VSOURCE" H 1328 2705 50  0000 L CNN
 F 2 "" H 1100 2750 50  0001 C CNN
@@
 $EndComp
 $Comp
-L pspice:0 #GND?
+L pspice:0 #GND0102
 U 1 1 5EC9EDCB
 P 1100 3200
-F 0 "#GND?" H 1100 3100 50  0001 C CNN
+F 0 "#GND0102" H 1100 3100 50  0001 C CNN
 F 1 "0" H 1100 3289 50  0000 C CNN
 F 2 "" H 1100 3200 50  0001 C CNN
@@
 	4350 4200 4350 4400
 $Comp
-L pspice:VSOURCE Vpulse
-U 1 1 5ECA3209
-P 4000 4750
-F 0 "Vpulse" H 4228 4796 50  0000 L CNN
-F 1 "VSOURCE" H 4228 4705 50  0000 L CNN
-F 2 "" H 4000 4750 50  0001 C CNN
-F 3 "~" H 4000 4750 50  0001 C CNN
-F 4 "V" H 4000 4750 50  0001 C CNN "Spice_Primitive"
-F 5 "dc 10 pulse(0 10 2.7u 100n 100n 1.2u 4.5u)" H 4000 4750 50  0001 C CNN "Spice_Model"
-F 6 "Y" H 4000 4750 50  0001 C CNN "Spice_Netlist_Enabled"
-	1    4000 4750
-	1    0    0    -1
-$EndComp
-$Comp
-L pspice:0 #GND?
+L pspice:0 #GND0103
 U 1 1 5ECA3644
 P 4000 5150
-F 0 "#GND?" H 4000 5050 50  0001 C CNN
+F 0 "#GND0103" H 4000 5050 50  0001 C CNN
 F 1 "0" H 4000 5239 50  0000 C CNN
 F 2 "" H 4000 5150 50  0001 C CNN
@@
 	4000 4000 4050 4000
 $Comp
-L pspice:R Rload
+L pspice:R Rload1
 U 1 1 5ECA69A3
 P 6350 2800
-F 0 "Rload" H 6418 2846 50  0000 L CNN
+F 0 "Rload1" H 6418 2846 50  0000 L CNN
 F 1 "R" H 6418 2755 50  0000 L CNN
 F 2 "" H 6350 2800 50  0001 C CNN
 F 3 "~" H 6350 2800 50  0001 C CNN
 F 4 "R" H 6350 2800 50  0001 C CNN "Spice_Primitive"
-F 5 "20" H 6350 2800 50  0001 C CNN "Spice_Model"
+F 5 "400" H 6350 2800 50  0001 C CNN "Spice_Model"
 F 6 "Y" H 6350 2800 50  0001 C CNN "Spice_Netlist_Enabled"
 	1    6350 2800
@@
 $EndComp
 $Comp
-L pspice:0 #GND?
+L pspice:0 #GND0104
 U 1 1 5ECA6E2B
 P 6350 3200
-F 0 "#GND?" H 6350 3100 50  0001 C CNN
+F 0 "#GND0104" H 6350 3100 50  0001 C CNN
 F 1 "0" H 6350 3289 50  0000 C CNN
 F 2 "" H 6350 3200 50  0001 C CNN
@@
 	6350 3050 6350 3200
 $Comp
-L pspice:C Cout
+L pspice:C Cout1
 U 1 1 5ECA86D5
 P 6700 2800
-F 0 "Cout" H 6878 2846 50  0000 L CNN
+F 0 "Cout1" H 6878 2846 50  0000 L CNN
 F 1 "C" H 6878 2755 50  0000 L CNN
 F 2 "" H 6700 2800 50  0001 C CNN
@@
 $EndComp
 $Comp
-L pspice:0 #GND?
+L pspice:0 #GND0105
 U 1 1 5ECA918F
 P 6700 3200
-F 0 "#GND?" H 6700 3100 50  0001 C CNN
+F 0 "#GND0105" H 6700 3100 50  0001 C CNN
 F 1 "0" H 6700 3289 50  0000 C CNN
 F 2 "" H 6700 3200 50  0001 C CNN
@@
 	6700 2550 6700 2350
 $Comp
-L pspice:R Rsource
+L pspice:R Rsource1
 U 1 1 5ECA420F
 P 4350 3450
-F 0 "Rsource" H 4418 3496 50  0000 L CNN
+F 0 "Rsource1" H 4418 3496 50  0000 L CNN
 F 1 "R" H 4418 3405 50  0000 L CNN
 F 2 "" H 4350 3450 50  0001 C CNN
@@
 	6350 2550 6350 2350
 $Comp
-L pspice:C Cmid
+L pspice:C Cmid1
 U 1 1 5EC9E1D7
 P 4000 2350
-F 0 "Cmid" V 3685 2350 50  0000 C CNN
+F 0 "Cmid1" V 3685 2350 50  0000 C CNN
 F 1 "C" V 3776 2350 50  0000 C CNN
 F 2 "" H 4000 2350 50  0001 C CNN
@@
 $EndComp
 $Comp
-L pspice:C Cmid?
+L pspice:C Cmid2
 U 1 1 5ECBC084
 P 4700 4050
-F 0 "Cmid?" V 4385 4050 50  0000 C CNN
+F 0 "Cmid2" V 4385 4050 50  0000 C CNN
 F 1 "C" V 4476 4050 50  0000 C CNN
 F 2 "" H 4700 4050 50  0001 C CNN
@@
 Connection ~ 4350 2350
 $Comp
-L pspice:0 #GND?
+L pspice:0 #GND0106
 U 1 1 5ECBFF1F
 P 4700 4400
-F 0 "#GND?" H 4700 4300 50  0001 C CNN
+F 0 "#GND0106" H 4700 4300 50  0001 C CNN
 F 1 "0" H 4700 4489 50  0000 C CNN
 F 2 "" H 4700 4400 50  0001 C CNN
@@
 $EndComp
 $Comp
-L pspice:VSOURCE Vpulse?
+L pspice:VSOURCE Vpulse1
 U 1 1 5ED498F6
 P 2850 2700
-F 0 "Vpulse?" H 3078 2746 50  0000 L CNN
+F 0 "Vpulse1" H 3078 2746 50  0000 L CNN
 F 1 "VSOURCE" H 3078 2655 50  0000 L CNN
 F 2 "" H 2850 2700 50  0001 C CNN
 F 3 "~" H 2850 2700 50  0001 C CNN
 F 4 "V" H 2850 2700 50  0001 C CNN "Spice_Primitive"
-F 5 "dc 10 pulse(0 10 0u 100n 100n 2.5u 4.5u)" H 2850 2700 50  0001 C CNN "Spice_Model"
+F 5 "dc 10 pulse(0 10 0u 100n 100n 1000n 3.5u)" H 2850 2700 50  0001 C CNN "Spice_Model"
 F 6 "Y" H 2850 2700 50  0001 C CNN "Spice_Netlist_Enabled"
 	1    2850 2700
@@
 Connection ~ 3150 2350
 $Comp
-L pspice:0 #GND?
+L pspice:0 #GND0107
 U 1 1 5ED638C3
 P 3300 3550
-F 0 "#GND?" H 3300 3450 50  0001 C CNN
+F 0 "#GND0107" H 3300 3450 50  0001 C CNN
 F 1 "0" H 3300 3639 50  0000 C CNN
 F 2 "" H 3300 3550 50  0001 C CNN
@@
 	5600 3200 5600 3050
 $Comp
-L pspice:0 #GND?
+L pspice:0 #GND0108
 U 1 1 5ECA2A97
 P 5600 3200
-F 0 "#GND?" H 5600 3100 50  0001 C CNN
+F 0 "#GND0108" H 5600 3100 50  0001 C CNN
 F 1 "0" H 5600 3289 50  0000 C CNN
 F 2 "" H 5600 3200 50  0001 C CNN
@@
 $EndComp
 $Comp
-L pspice:DIODE Drect
+L pspice:DIODE Drect1
 U 1 1 5ECAA3B0
 P 5200 1250
-F 0 "Drect" H 5200 1515 50  0000 C CNN
+F 0 "Drect1" H 5200 1515 50  0000 C CNN
 F 1 "DIODE" H 5200 1424 50  0000 C CNN
 F 2 "" H 5200 1250 50  0001 C CNN
@@
 	5600 2350 6350 2350
 $Comp
-L pspice:0 #GND?
+L pspice:0 #GND0109
 U 1 1 5EDA40EF
 P 5200 1450
-F 0 "#GND?" H 5200 1350 50  0001 C CNN
+F 0 "#GND0109" H 5200 1350 50  0001 C CNN
 F 1 "0" H 5200 1539 50  0000 C CNN
 F 2 "" H 5200 1450 50  0001 C CNN
@@
 	4350 2350 4350 3200
 $Comp
-L pspice:INDUCTOR Lout
+L pspice:INDUCTOR Lout1
 U 1 1 5ECA22CE
 P 5050 2350
-F 0 "Lout" V 5004 2428 50  0000 L CNN
+F 0 "Lout1" V 5004 2428 50  0000 L CNN
 F 1 "INDUCTOR" V 5095 2428 50  0000 L CNN
 F 2 "" H 5050 2350 50  0001 C CNN
@@
 $EndComp
 $Comp
-L pspice:INDUCTOR Lin
+L pspice:INDUCTOR Lin1
 U 1 1 5EC9CFEB
 P 3300 3250
-F 0 "Lin" H 3300 3465 50  0000 C CNN
+F 0 "Lin1" H 3300 3465 50  0000 C CNN
 F 1 "INDUCTOR" H 3300 3374 50  0000 C CNN
 F 2 "" H 3300 3250 50  0001 C CNN
@@
 Text Notes 1400 5550 0    50   ~ 0
 Note: This can really scarf down amps... Need a lot of input capacitance.
+$Comp
+L pspice:VSOURCE Vpulse2
+U 1 1 5ECA3209
+P 4000 4750
+F 0 "Vpulse2" H 4228 4796 50  0000 L CNN
+F 1 "VSOURCE" H 4228 4705 50  0000 L CNN
+F 2 "" H 4000 4750 50  0001 C CNN
+F 3 "~" H 4000 4750 50  0001 C CNN
+F 4 "V" H 4000 4750 50  0001 C CNN "Spice_Primitive"
+F 5 "dc 10 pulse(0 0 900n 100n 100n 700n 2.1u)" H 4000 4750 50  0001 C CNN "Spice_Model"
+F 6 "Y" H 4000 4750 50  0001 C CNN "Spice_Netlist_Enabled"
+	1    4000 4750
+	1    0    0    -1
+$EndComp
 $EndSCHEMATC
