File: multitool/multitool.sch (KiCad schematic (older format))
At the start: 75 parts, among them J1 USB_B_Micro, J10 TPI, J11 UPDI, J12 UNIVERSAL, J13 PGMIF, J14 Conn_01x04, J2 JTAG, J3 PGMIF, J4 WSOUT, J5 VPPS, J6 SAO, J7 VDDS, J8 PADAUK, J9 AVR, Q1 3404, Q2 3404, Q3 3404, Q4 3404, Q5 Q_PNP_BEC, Q6 3404, Q7 3404, SW1 BOOT0, U1 STM32F042F4Px, U2 MT2492, U3 NUP4202, U4 XC6206P360MR, U5 EG27324, U6 INA181A3

Commit message: Add untested note
Other:
- note added: "DRAFT NOT FOR MANUFACTURE"
Changed lines of the file:
@@
 Wire Wire Line
 	10450 2300 10900 2300
+Text Notes 6700 6950 0    197  ~ 0
+DRAFT NOT FOR MANUFACTURE
 $EndSCHEMATC

Commit message: Getting closer
Parts:
- removed J11: UPDI, Connector_PinSocket_2.54mm:PinSocket_2x03_P2.54mm_Vertical_SMD, symbol Connector_Generic:Conn_02x03_Odd_Even
- added J15: ESP-01, Connector_PinSocket_2.54mm:PinSocket_2x04_P2.54mm_Vertical_SMD, symbol Connector_Generic:Conn_02x04_Odd_Even
- added J16: VDDS, Jumper:SolderJumper-2_P1.3mm_Bridged_Pad1.0x1.5mm, symbol Connector_Generic:Conn_01x02
- added J17, J18, J19, J20: MNT, MountingHole:MountingHole_5.3mm_M5_Pad_Via, symbol Connector_Generic:Conn_01x01
- J13: value PGMIF -> PG4
- J14: value Conn_01x04 -> WS2813
- J2: value JTAG -> SELF_PGM
- J3: value PGMIF -> PGDA
Connections:
- net +3V8: now also J16.1 (Pin_1), J16.2 (Pin_2); no longer J5.1 (Pin_1), J7.1 (Pin_1)
- net GND: now also J15.1 (Pin_1), J17.1 (Pin_1), J18.1 (Pin_1), J19.1 (Pin_1), J20.1 (Pin_1)
- net PD_VDD: now also J15.8 (Pin_8)
- net PD_VPP: now also J15.6 (Pin_6)
- net SCL: now also J15.3 (Pin_3)
- net SDA: now also J15.5 (Pin_5)
- net U2CK: now also J15.4 (Pin_4)
- net U2RX: now also J15.2 (Pin_2)
- net U2TX: now also J15.7 (Pin_7)
- net VUSB: now also J5.1 (Pin_1), J7.1 (Pin_1)
Other:
- note added: "Also force PD_VPP low.\n(default)"
- note removed: "Also force PD_VPP low."
- note removed: "from microUPDI"
- moved on the sheet: C19, D1, D2, Q3, R14, R9, U4

Commit message: bump
Other:
- note added: "TODO: Use Zeta - and probably EG3012 or EG3013 (Good to 4.5v) Maybe EG3112 (HIN/LIN) or EG2104, EG2130 (IN/SD) (Good to lower voltage)"
- note removed: "TODO: For Padauk, should magic be on TX or RX?"
- moved on the sheet: C11, C12, C13, C14, C15, C19, C9, D1, D2, J10, J12, J13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

Commit message: update some tweaks to the zeta sim thoughts.
Parts:
- removed C1, C26: 2.2uF, Capacitor_SMD:C_0805_2012Metric_Pad1.15x1.40mm_HandSolder, symbol multitool-rescue:C-Device-tensigral_lamp_hardware-rescue-tensigral_lamp_hardwar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
- removed C14, C15, C17, C9: 22nF, Capacitor_SMD:C_0805_2012Metric_Pad1.15x1.40mm_HandSolder, symbol multitool-rescue:C-Device-tensigral_lamp_hardware-rescue-tensigral_lamp_hardwar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
- removed D21, D22: 1N4002, Diode_SMD:D_SOD-123F, symbol Device:D
- removed J3: PGDA, Jumper:SolderJumper-3_P1.3mm_Bridged12_RoundedPad1.0x1.5mm, symbol Connector_Generic:Conn_01x03
- removed Q1, Q2, Q6, Q7: 3404, Package_TO_SOT_SMD:SOT-23, symbol Device:Q_NMOS_GSD
- removed R10, R12, R14, R9: 680, Resistor_SMD:R_0805_2012Metric_Pad1.15x1.40mm_HandSolder, symbol multitool-rescue:R-Device-tensigral_lamp_hardware-rescue-tensigral_lamp_hardwar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
- removed R11, R13, R5, R6, R7, R8: 220, Resistor_SMD:R_0805_2012Metric_Pad1.15x1.40mm_HandSolder, symbol multitool-rescue:R-Device-tensigral_lamp_hardware-rescue-tensigral_lamp_hardwar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
- removed R16, R19: 1k, Resistor_SMD:R_0805_2012Metric_Pad1.15x1.40mm_HandSolder, symbol multitool-rescue:R-Device-tensigral_lamp_hardware-rescue-tensigral_lamp_hardwar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
- removed U1: STM32F042F4Px, Package_SO:TSSOP-20_4.4x6.5mm_P0.65mm, symbol multitool-rescue:STM32F042F4Px-MCU_ST_STM32F0-tensigral_lamp_hardware-rescue-te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
- added C?: 10u25v, Capacitor_SMD:C_0805_2012Metric_Pad1.15x1.40mm_HandSolder, symbol multitool-rescue:C-Device-tensigral_lamp_hardware-rescue-tensigral_lamp_hardwar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
- added C? (x5): 22nF, Capacitor_SMD:C_0603_1608Metric, symbol multitool-rescue:C-Device-tensigral_lamp_hardware-rescue-tensigral_lamp_hardwar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
- added Q? (x4): 3402, Package_TO_SOT_SMD:SOT-23, symbol Device:Q_NMOS_GSD
- added R? (x2): 680, Resistor_SMD:R_0805_2012Metric_Pad1.15x1.40mm_HandSolder, symbol multitool-rescue:R-Device-tensigral_lamp_hardware-rescue-tensigral_lamp_hardwar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
- added R? (x6): 1k, Resistor_SMD:R_0603_1608Metric, symbol multitool-rescue:R-Device-tensigral_lamp_hardware-rescue-tensigral_lamp_hardwar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
- added R? (x2): 330, Resistor_SMD:R_0603_1608Metric, symbol multitool-rescue:R-Device-tensigral_lamp_hardware-rescue-tensigral_lamp_hardwar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
- added R? (x5): 100, Resistor_SMD:R_0603_1608Metric, symbol multitool-rescue:R-Device-tensigral_lamp_hardware-rescue-tensigral_lamp_hardwar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
- added U? (x2): NCE2003, symbol NCE2003:NCE2003
- added U?: STM32F042K4Tx, Package_QFP:LQFP-32_7x7mm_P0.8mm, symbol MCU_ST_STM32F0:STM32F042K4Tx
- C11: footprint Capacitor_SMD:C_0805_2012Metric_Pad1.15x1.40mm_HandSolder -> Capacitor_SMD:C_0603_1608Metric; Cost100 0.003738 -> 0.003; LCSC https://lcsc.com/product-detail/Multilayer-Ceramic-Capacitors-MLCC-SMD-SMT_Walsin-Tech-Corp-0805B223K500_C123617.html -> https://lcsc.com/product-detail/Multilayer-Ceramic-Capacitors-MLCC-SMD-SMT_Walsin-Tech-Corp-0603B223K500_C123507.html
- C25: value 2.2uF -> 10u25v; Cost100 0.011787 -> 0.017645; LCSC https://lcsc.com/product-detail/Multilayer-Ceramic-Capacito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 -> https://lcsc.com/product-detail/New-Arrivals_Taiyo-Yuden-TM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
- J1: value USB_B_Micro -> USB
- Q4: value 3404 -> 3402; Cost100 0.023864 -> 0.025; LCSC https://lcsc.com/product-detail/MOSFET_Wuxi-NCE-Power-Semic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 -> https://lcsc.com/product-detail/MOSFET_Guangdong-Hottech-AO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
- R1: footprint Resistor_SMD:R_0805_2012Metric_Pad1.15x1.40mm_HandSolder -> Resistor_SMD:R_0603_1608Metric; Cost100 0.002409 -> 0.002; LCSC https://lcsc.com/product-detail/Chip-Resistor-Surface-Mount_UNI-ROYAL-Uniroyal-Elec-0805W8F2702T5E_C17593.html -> https://lcsc.com/product-detail/Chip-Resistor-Surface-Mount_UNI-ROYAL-Uniroyal-Elec-0603WAF2702T5E_C22967.html
- R15: footprint Resistor_SMD:R_0805_2012Metric_Pad1.15x1.40mm_HandSolder -> Resistor_SMD:R_0603_1608Metric; Cost100 0.002315 -> 0.002; LCSC https://lcsc.com/product-detail/Chip-Resistor-Surface-Mount_UNI-ROYAL-Uniroyal-Elec-0805W8F1001T5E_C17513.html -> https://lcsc.com/product-detail/Chip-Resistor-Surface-Mount_UNI-ROYAL-Uniroyal-Elec-0603WAF1001T5E_C21190.html
- R18, R2: footprint Resistor_SMD:R_0805_2012Metric_Pad1.15x1.40mm_HandSolder -> Resistor_SMD:R_0603_1608Metric; Cost100 0.002315 -> 0.002; LCSC https://lcsc.com/product-detail/Chip-Resistor-Surface-Mount_UNI-ROYAL-Uniroyal-Elec-0805W8F4701T5E_C17673.html -> https://lcsc.com/product-detail/Chip-Resistor-Surface-Mount_UNI-ROYAL-Uniroyal-Elec-0603WAF4701T5E_C23162.html
- R3: value 4.7k-1% -> 4.7k; footprint Resistor_SMD:R_0805_2012Metric_Pad1.15x1.40mm_HandSolder -> Resistor_SMD:R_0603_1608Metric; Cost100 0.002315 -> 0.002; LCSC https://lcsc.com/product-detail/Chip-Resistor-Surface-Mount_UNI-ROYAL-Uniroyal-Elec-0805W8F4701T5E_C17673.html -> https://lcsc.com/product-detail/Chip-Resistor-Surface-Mount_UNI-ROYAL-Uniroyal-Elec-0603WAF4701T5E_C23162.html
- R4: value 220 -> 100; footprint Resistor_SMD:R_0805_2012Metric_Pad1.15x1.40mm_HandSolder -> Resistor_SMD:R_0603_1608Metric; Cost100 0.00229 -> 0.002; LCSC https://lcsc.com/product-detail/Chip-Resistor-Surface-Mount_UNI-ROYAL-Uniroyal-Elec-0805W8F2200T5E_C17557.html -> https://lcsc.com/product-detail/Chip-Resistor-Surface-Mount_UNI-ROYAL-Uniroyal-Elec-0603WAF1000T5E_C22775.html
Connections:
- net +3V3: now also U?.1 (VDD), U?.17 (VDDIO2)
- net +3V8: now also C?.1
- net AVCC: now also C?.1, C?.1, U?.5 (VDDA)
- net D+: now also U?.22 (PA12)
- net D-: now also U?.21 (PA11)
- net GND: now also L3.2, L4.2, C?.2, C?.2, C?.2, C?.2, C?.2, C?.2, Q?.2 (S), Q?.2 (S), Q?.2 (S), Q?.2 (S), R?.2, R?.2, R?.2, R?.2, U?.16 (VSS), U?.32 (VSSA), U?.5 (S1), U?.5 (S1); no longer L5.2, L6.2
- net MAGICPIN: now also Q?.3 (D), R?.1
- net MPMON: now also R?.1, U?.15 (PB1)
- net NRST: now also C?.1, U?.4 (NRST)
- net PD_VDD: now also R?.1
- net PD_VPP: now also L5.2, Q?.3 (D), R?.1
- net PIMON: now also U?.14 (PB0)
- net SCL: now also R?.1
- net SWC: now also U?.24 (PA14)
- net SWD: now also Q?.1 (G), U?.23 (PA13)
- net U2CK: now also R?.1
- net U2RTS: now also U?.7 (PA1)
- net U2RX: now also R?.1; no longer J10.4 (Pin_4)
- net U2RXDIRECT: now also R?.2, R?.2, U?.9 (PA3)
- net U2TX: now also J8.5 (Pin_5), R?.1
- net VMON1: now also R?.1, R?.2, U?.6 (PA0)
- net VMON2: now also R?.1, R?.2, U?.11 (PA5)
- net VUSB: now also C?.1; no longer J5.1 (Pin_1)
- net WS2812: now also J10.4 (Pin_4), U?.13 (PA7)
- net at R4.2: now also U?.2 (PF0)
- net at R17.1, U6.3 (+): now also L6.2, C?.1
- net at L3.1: now also C23.2, U?.4 (D2); no longer J5.2 (Pin_2)
- net at C23.1, L5.1: now also Q?.3 (D)
- net at U5.5 (OUTB): now also Q?.1 (G)
- net at J7.2 (Pin_2): now also R?.1, U?.2 (S2); no longer L4.1
- net at C24.2: now also L4.1, U?.4 (D2); no longer L4.2
- net at C24.1, L6.1: now also Q?.3 (D)
- net at Q3.3 (D): now also R?.2
- net at D1.1 (K): now also R?.1
- net at D2.1 (K): now also R?.1
- net TIM16_CH1: no longer names the net of R3.2, SW1.4
- net TIM16_CH1: now also U?.31 (PB8)
- new net: R?.2, U?.3 (G2), U?.6 (D1) (x2)
- new net: R?.2, U?.10 (PA4)
- new net: R?.2, U?.3 (PF1)
- new net: J5.2 (Pin_2), R?.1, U?.2 (S2)
- new net SW1VDD: U?.1 (G1)
- new net SW1VPP: U?.1 (G1)
- new net SW2VDD: Q?.1 (G)
- new net SW2VPP: Q?.1 (G)
- new net T3C1: U?.27 (PB4)
- new net T3C2: U?.28 (PB5)
- new net U1CK: U?.18 (PA8)
- new net U1RX: U?.30 (PB7)
- new net U1TX: R?.2
- new net U1TXCOMB: R?.1, U?.20 (PA10), U?.29 (PB6)
- new net U2RCOMB: R?.2, U?.25 (PA15), U?.8 (PA2)
Other:
- note added: "Does USART have SPI mode?\nDo we need UART1? \nCan use a buffer to the UART1 RX pin?"
- note added: "Supports\n * PDI\n * JTAG\n * SWD"
- note added: "TODO: USE LINE DRIVER FOR RX"
- note added: "TODO:\nSplit out SPI\nWhat devices would prefer SPI?"
- note removed: "Also, should be able to be:\n * PDI\n * JTAG\n * SWD"
- note removed: "TODO: Use Zeta - and probably EG3012 or EG3013 (Good to 4.5v) Maybe EG3112 (HIN/LIN) or EG2104, EG2130 (IN/SD) (Good to lower voltage)"
- moved on the sheet: C11, C23, C24, C25, D1, D2, D3, D4, D5, J10, J12, J14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

Commit message: Tweak multitool design.
Parts:
- removed C12, C13, C16: 22uF, Capacitor_SMD:C_0805_2012Metric_Pad1.15x1.40mm_HandSolder, symbol multitool-rescue:C-Device-tensigral_lamp_hardware-rescue-tensigral_lamp_hardwar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
- removed J10: TPI, Connector_PinSocket_2.54mm:PinSocket_2x03_P2.54mm_Vertical_SMD, symbol Connector_Generic:Conn_02x03_Odd_Even
- removed J13: PG4, Jumper:SolderJumper-3_P1.3mm_Bridged12_RoundedPad1.0x1.5mm, symbol Connector_Generic:Conn_01x03
- removed J8: PADAUK, Connector_PinSocket_2.54mm:PinSocket_2x04_P2.54mm_Vertical_SMD, symbol Connector_Generic:Conn_02x04_Odd_Even
- removed Q?: 3402, Package_TO_SOT_SMD:SOT-23, symbol Device:Q_NMOS_GSD
- removed R18: 4.7k, Resistor_SMD:R_0603_1608Metric, symbol multitool-rescue:R-Device-tensigral_lamp_hardware-rescue-tensigral_lamp_hardwar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
- removed R?: 100, Resistor_SMD:R_0603_1608Metric, symbol multitool-rescue:R-Device-tensigral_lamp_hardware-rescue-tensigral_lamp_hardwar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
- removed R?: 1k, Resistor_SMD:R_0603_1608Metric, symbol multitool-rescue:R-Device-tensigral_lamp_hardware-rescue-tensigral_lamp_hardwar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
- removed U5: EG27324, Package_SO:SO-8_3.9x4.9mm_P1.27mm, symbol EG27324:EG27324
- added C? (x3): 10u25v, Capacitor_SMD:C_0805_2012Metric_Pad1.15x1.40mm_HandSolder, symbol multitool-rescue:C-Device-tensigral_lamp_hardware-rescue-tensigral_lamp_hardwar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
- added J?: PADAUK, Connector_PinSocket_2.54mm:PinSocket_2x05_P2.54mm_Vertical_SMD, symbol Connector_Generic:Conn_02x05_Odd_Even
- added R? (x2): 100, Resistor_SMD:R_0603_1608Metric, symbol multitool-rescue:R-Device-tensigral_lamp_hardware-rescue-tensigral_lamp_hardwar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
- added R?: 4.7k, Resistor_SMD:R_0603_1608Metric, symbol multitool-rescue:R-Device-tensigral_lamp_hardware-rescue-tensigral_lamp_hardwar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
- added R? (x2): 1k, Resistor_SMD:R_0603_1608Metric, symbol multitool-rescue:R-Device-tensigral_lamp_hardware-rescue-tensigral_lamp_hardwar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
- added R?: 27k, Resistor_SMD:R_0603_1608Metric, symbol multitool-rescue:R-Device-tensigral_lamp_hardware-rescue-tensigral_lamp_hardwar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
- added U?: 74LVC02APW, Package_SO:TSSOP-14_4.4x5mm_P0.65mm, symbol Interface_UART:ST485EBDR
- added U? (x5): 74LVC02APW, Package_SO:TSSOP-14_4.4x5mm_P0.65mm, symbol 74xx:7402
- D4: value 3.1V Zener -> 3.6V; Cost100 .008013 -> 0.084843; LCSC https://lcsc.com/product-detail/Zener-Diodes_Shandong-Jingd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 -> https://lcsc.com/product-detail/Zener-Diodes_Vishay-Interte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
- J12: footprint Connector_PinSocket_2.54mm:PinSocket_2x05_P2.54mm_Vertical_SMD -> Connector_PinHeader_2.54mm:PinHeader_2x05_P2.54mm_Vertical_SMD
- U? (x2): value NCE2003 -> 74LVC02APW; footprint (none) -> Package_SO:TSSOP-14_4.4x5mm_P0.65mm
- U?: value STM32F042K4Tx -> 74LVC02APW; footprint Package_QFP:LQFP-32_7x7mm_P0.8mm -> Package_SO:TSSOP-14_4.4x5mm_P0.65mm
Connections:
- net MPMON is gone; now on net SW2VDD: U?.15 (PB1)
- net T3C2 is gone; now on an unnamed net: U?.28 (PB5)
- net U1CK is gone; now on net SW1VPP: U?.18 (PA8)
- net +3V3: now also U?.14 (VCC)
- net +3V8: now also C?.1
- net AVCC: now also C?.1
- net GND: now also J6.2 (Pin_2), J9.6 (Pin_6), C?.2, C?.2, C?.2, J?.3 (Pin_3), R?.1, R?.1, U?.5 (GND), U?.7 (GND); no longer J6.1 (Pin_1), J9.5 (Pin_5)
- net MAGICPIN: now also J12.8 (Pin_8), J9.5 (Pin_5), J?.10 (Pin_10), R?.1; no longer J12.7 (Pin_7)
- net PD_VDD: now also J12.10 (Pin_10), J6.1 (Pin_1), J9.2 (Pin_2), J?.4 (Pin_4); no longer J12.5 (Pin_5), J6.2 (Pin_2), J9.1 (Pin_1)
- net PD_VPP: now also R?.1, R?.2; no longer J9.6 (Pin_6)
- net PIMON: now also U?.13 (PA7); no longer U?.14 (PB0)
- net SCL: now also J6.4 (Pin_4), J?.6 (Pin_6); no longer J12.4 (Pin_4), J6.3 (Pin_3)
- net SDA: now also J6.3 (Pin_3); no longer J12.3 (Pin_3), J6.4 (Pin_4)
- net SW1VDD: now also U?.14 (PB0)
- net SW1VPP: now also R?.2, R?.2
- net SW2VPP: now also U?.19 (PA9)
- net U2CK: no longer J12.6 (Pin_6), J9.4 (Pin_4)
- net U2RTS: now also J12.6 (Pin_6), U?.2, U?.3, U?.6, U?.9
- net U2RX: now also D4.1 (K), J6.6 (Pin_6), R?.2, J?.5 (Pin_5), U?.1 (RO); no longer J12.10 (Pin_10), J6.5 (Pin_5), J9.2 (Pin_2)
- net U2TX: now also J6.5 (Pin_5), U?.11, U?.12, U?.4 (DI), U?.5; no longer J12.8 (Pin_8), J6.6 (Pin_6), J9.3 (Pin_3)
- net VUSB: now also J12.3 (Pin_3), J5.1 (Pin_1), C?.1, U?.8 (VCC)
- net at U?.12 (PA6): now also R?.2
- net SPISCK: now reaches U?.26 (PB3)
- net SPISCK: now also J9.3 (Pin_3), J?.9 (Pin_9)
- net DRIVEHI: now reaches Q4.1 (G)
- net DRIVEHI: now also U?.10
- net DRIVELO: now reaches Q?.1 (G)
- net DRIVELO: now also U?.4
- net at Q5.1 (B), R15.1: now also R?.2
- net T3C1: no longer names the net of U?.27 (PB4)
- net T3C1: now also R?.1
- net U1RX: no longer names the net of U?.30 (PB7)
- net U1TXCOMB: no longer names the net of U?.20 (PA10)
- net U1TXCOMB: no longer U?.29 (PB6)
- net U2RCOMB: no longer names the net of R?.2, U?.8 (PA2)
- net U2RCOMB: now also U?.9 (PA3); no longer U?.25 (PA15)
- removed net U2RXDIRECT: D4.1 (K), R?.2, R?.2, U?.9 (PA3)
- net WS2812 renamed SPIMOSICOMB
- net SPIMOSICOMB: now also J9.1 (Pin_1), J?.8 (Pin_8), R?.2; no longer U?.13 (PA7)
- new net: R?.2, U?.25 (PA15)
- new net 485A: J12.7 (Pin_7), U?.6 (A)
- new net 485B: J12.5 (Pin_5), U?.7 (B)
- new net SPIMISO: J12.4 (Pin_4), J9.4 (Pin_4), J?.7 (Pin_7), R?.1
- new net U2TXEN: U?.1, U?.3 (DE)
- new net ~485RXEN~: U?.2 (~RE), U?.29 (PB6)
- new net ~U2TX~: U?.13, U?.8
- no-connect marks 0 -> 2
Other:
- note added: "AVR ISP/TPI/UPDI"
- note added: "Base R is not needed if PNP"
- note added: "G1"
- note added: "G2"
- note added: "ICVPP/PA5"
- note added: "IPDA/PA6"
- note added: "OK"
- note added: "PA3/IPCK"
- note added: "PDI/ESP/Serial"
- note added: "Probably SWIM + SWD"
- note added: "RS-485, DMX-512 too!"
- note added: "SAO/Imon/I2C"
- note added: "T16_CH1 Alt"
- note added: "T1C1\nT1C2"
- note added: "T2CH2 ALT"
- note added: "T2CH3 ALT"
- note added: "T3C3\nT3C4"
- note added: "U2TX alt is TIM2_CH3"
- note added: "U2TX can also function as SPI_NSS"
- note removed: "Also force PD_VPP low.\n(default)"
- note removed: "Does USART have SPI mode?\nDo we need UART1? \nCan use a buffer to the UART1 RX pin?"
- note removed: "ICVPP"
- note removed: "IPCK / U2CK\n"
- note removed: "IPDA / U2TX"
- note removed: "Supports\n * PDI\n * JTAG\n * SWD"
- note removed: "TODO:\nSplit out SPI\nWhat devices would prefer SPI?"
- moved on the sheet: C23, C24, C25, C?, D23, D5, J12, J15, J16, J4, J5, J6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

Commit message: Bump
Parts:
- removed J12: UNIVERSAL, Connector_PinHeader_2.54mm:PinHeader_2x05_P2.54mm_Vertical_SMD, symbol Connector_Generic:Conn_02x05_Odd_Even
- removed Q3: 3404, Package_TO_SOT_SMD:SOT-23, symbol Device:Q_NMOS_GSD
- removed R?: 100, Resistor_SMD:R_0603_1608Metric, symbol multitool-rescue:R-Device-tensigral_lamp_hardware-rescue-tensigral_lamp_hardwar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
- added D6: BLU, LED_SMD:LED_0805_2012Metric_Pad1.15x1.40mm_HandSolder, symbol Device:LED
- added D7: 5.1V, Diode_SMD:D_SOD-123, symbol Device:D_Zener
- added J3: UNIVERSAL, Connector_PinHeader_2.54mm:PinHeader_2x07_P2.54mm_Vertical_SMD, symbol Connector_Generic:Conn_02x07_Odd_Even
- added R11: 1k, Resistor_SMD:R_0603_1608Metric, symbol multitool-rescue:R-Device-tensigral_lamp_hardware-rescue-tensigral_lamp_hardwar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
- added SW2: SUBCFG, kicad:TACTILE10B, symbol multitool-rescue:TACTILE-tactile-tensigral_lamp_hardware-rescue-tensigral_lamp_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
- D1: value LED -> RED
- D2: value LED -> GRN; Cost100 .00889 -> .0103; LCSC https://lcsc.com/product-detail/Light-Emitting-Diodes-LED_0805_C205444.html -> https://lcsc.com/product-detail/Light-Emitting-Diodes-LED_0805-green_C205442.html
- D4: value 3.6V -> 5.1V; Cost100 0.084843 -> 0.01; LCSC https://lcsc.com/product-detail/Zener-Diodes_Vishay-Interte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 -> https://lcsc.com/product-detail/Zener-Diodes_Shandong-Jingd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
- U1: renamed from U?; value 74LVC02APW -> STM32F042; footprint Package_SO:TSSOP-14_4.4x5mm_P0.65mm -> Package_QFP:TQFP-32_7x7mm_P0.8mm
- U5: renamed from U?; value 74LVC02APW -> SP485; footprint Package_SO:TSSOP-14_4.4x5mm_P0.65mm -> Package_SO:SOP-8_3.9x4.9mm_P1.27mm
- U8, U9: renamed from U?; value 74LVC02APW -> LOADSW; footprint Package_SO:TSSOP-14_4.4x5mm_P0.65mm -> Package_TO_SOT_SMD:SOT-23-6
- gave numbers to parts that had none: 32
Connections:
- net +3V3: now also D1.2 (A), D6.2 (A)
- net +3V8: now also SW2.1; no longer D1.2 (A)
- net 485A: now also J3.11 (Pin_11)
- net 485B: now also J3.9 (Pin_9)
- net GND: now also D7.2 (A), J3.1 (Pin_1), J3.13 (Pin_13), J3.2 (Pin_2); no longer D3.6 (BIN)
- net MAGICPIN: now also J3.14 (Pin_14)
- net PD_VDD: now also J3.4 (Pin_4); no longer R23.1
- net PD_VPP: now also J3.12 (Pin_12)
- net SDA: now also J8.5 (Pin_5)
- net SPIMISO: now also R11.2
- net SPISCK: now also D7.1 (K), J3.6 (Pin_6)
- net SWD: now also J3.7 (Pin_7)
- net U2RTS: now also J3.10 (Pin_10)
- net U2RX: now also J8.1 (Pin_1), R7.2, U1.25 (PA15), J3.8 (Pin_8); no longer J8.5 (Pin_5)
- net U2TX: now also J8.2 (Pin_2), J3.5 (Pin_5)
- net VUSB: now also J3.3 (Pin_3)
- net PA10: now reaches U1.20 (PA10)
- net PA10: now also D3.6 (BIN)
- net at U1.30 (PB7): now also SW2.4
- net at C9.1, L6.2, R17.1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: now also R23.1
- new net: D6.1 (K), R11.1
- no-connect marks 2 -> 0
Other:
- note added: "2x Servo, RS-485, DMX-512, IROUT"
- note added: "AVR ISP/TPI/UPDI + SWIM/SWD + SERVO"
- note added: "FEMALE"
- note added: "MALE"
- note added: "PADAUK, LCD, OLED, SPI FLASH"
- note added: "PDI/ESP/TTL Serial"
- note added: "T16CH1 ALT"
- note added: "T2CH2"
- note added: "T2CH3"
- note added: "U2TX can also function as SPI_NSS\nU2RX is 5V tolerant\nSPISCK is 5V tolerant"
- note removed: "AVR ISP/TPI/UPDI"
- note removed: "OK"
- note removed: "PDI/ESP/Serial"
- note removed: "Probably SWIM + SWD"
- note removed: "RS-485, DMX-512 too!"
- note removed: "T16_CH1 Alt"
- note removed: "T2CH2 ALT"
- note removed: "TODO: USE LINE DRIVER FOR RX"
- note removed: "U2TX can also function as SPI_NSS"
- moved on the sheet: C11, C7, C8, D1, D2, D4, D5, J2, J8, L1, Q3, Q4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
