File: multitool/multitool.kicad_pcb (KiCad board)
At the start: 2 copper layers, 75 parts, among them J1 USB_B_Micro, J10 TPI, J11 UPDI, J12 UNIVERSAL, J13 PGMIF, J14 Conn_01x04, J2 JTAG, J3 PGMIF, J4 WSOUT, J5 VPPS, J6 SAO, J7 VDDS, J8 PADAUK, J9 AVR, Q1 3404, Q2 3404, Q3 3404, Q4 3404, Q5 Q_PNP_BEC, Q6 3404, Q7 3404, SW1 BOOT0, U1 STM32F042F4Px, U2 MT2492, U3 NUP4202, U4 XC6206P360MR, U5 EG27324, U6 INA181A3

Commit message: Add untested note
Other:
- board text added: "UNTESTED"
Changed lines of the file:
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@@
   (general
     (thickness 1.6)
-    (drawings 7)
+    (drawings 8)
     (tracks 0)
     (zones 0)
@@
     )
   )
+  (gr_text UNTESTED (at 221.996 30.48) (layer F.Fab)
+    (effects (font (size 10 10) (thickness 1)))
+  )
   (gr_circle (center 47.16 56.925) (end 47.46 56.975) (layer F.SilkS) (width 0.12))

Commit message: Getting closer
Parts:
- removed J11: UPDI, Connector_PinSocket_2.54mm:PinSocket_2x03_P2.54mm_Vertical_SMD
- added J15: ESP-01, Connector_PinSocket_2.54mm:PinSocket_2x04_P2.54mm_Vertical_SMD, F.Cu at (130.8, 174.0)
- added J16: VDDS, Jumper:SolderJumper-2_P1.3mm_Bridged_Pad1.0x1.5mm, F.Cu at (124.5, 184.2)
- added J17: MNT, MountingHole:MountingHole_5.3mm_M5_Pad_Via, F.Cu at (86.4, 102.9)
- added J18: MNT, MountingHole:MountingHole_5.3mm_M5_Pad_Via, F.Cu at (142.2, 102.9)
- added J19: MNT, MountingHole:MountingHole_5.3mm_M5_Pad_Via, F.Cu at (142.2, 185.4)
- added J20: MNT, MountingHole:MountingHole_5.3mm_M5_Pad_Via, F.Cu at (86.4, 185.4)
- J13: value PGMIF -> PG4
- J14: value Conn_01x04 -> WS2813
- J2: value JTAG -> SELF_PGM
- J3: value PGMIF -> PGDA
- moved J12 170.5 mm to (86.4, 168.9)
- moved J3 150.0 mm to (109.2, 186.7), turned to 180 degrees
- moved J10 147.5 mm to (118.1, 185.4)
- moved J8 140.0 mm to (101.6, 184.2)
- moved L6 134.8 mm to (142.2, 115.6), turned to 90 degrees
- moved D22 134.1 mm to (142.2, 132.1), turned to 90 degrees
- moved C1 132.2 mm to (109.2, 165.1)
- moved C26 132.1 mm to (137.2, 129.5), turned to 180 degrees
- moved R10 130.0 mm to (120.7, 168.9), turned to 0 degrees
- moved J6 123.3 mm to (101.6, 157.5)
- moved D23 122.6 mm to (95.2, 153.7), turned to 90 degrees
- moved R11 122.3 mm to (115.6, 168.9), turned to 0 degrees
- moved D1 121.8 mm to (118.1, 149.9), turned to 270 degrees
- moved J13 121.8 mm to (109.2, 177.8), turned to 90 degrees
- moved R12 121.0 mm to (110.5, 154.9), turned to 180 degrees
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Connections:
- J5 pad 1: +3V8 -> VUSB
- J7 pad 1: +3V8 -> VUSB
Other:
- board outline added: 68.6 x 95.3 mm
- board text added: "0V DI 5V"
- board text added: "0V DI BI 5V"
- board text added: "ETX GND ENA GP2 RST GP0 VCC ERX"
- board text added: "GND VDD SDA SCL DX DAT CLK PGM"
- board text added: "NPX VPP SCL SDA UCK VDD DRX MAG DTX GND"
- board text added: "VDD ARX ATX UCK GND VPP"
- board text added: "VDD GND SDA SCL GP1 GP2"
- board text added: "VDD MISO MOSI SCK GND RST"

Commit message: Bump
Parts:
- removed C12, C13, C16: 22uF, Capacitor_SMD:C_0805_2012Metric_Pad1.15x1.40mm_HandSolder
- removed C14, C15, C17: 22nF, Capacitor_SMD:C_0805_2012Metric_Pad1.15x1.40mm_HandSolder
- removed C26: 2.2uF, Capacitor_SMD:C_0805_2012Metric_Pad1.15x1.40mm_HandSolder
- removed D21, D22: 1N4002, Diode_SMD:D_SOD-123F
- removed J10: TPI, Connector_PinSocket_2.54mm:PinSocket_2x03_P2.54mm_Vertical_SMD
- removed J12: UNIVERSAL, Connector_PinSocket_2.54mm:PinSocket_2x05_P2.54mm_Vertical_SMD
- removed J13: PG4, Jumper:SolderJumper-3_P1.3mm_Bridged12_RoundedPad1.0x1.5mm
- removed Q6, Q7: 3404, Package_TO_SOT_SMD:SOT-23
- added C2: 22nF, Capacitor_SMD:C_0603_1608Metric, F.Cu at (189.3, 84.1)
- added C3: 22nF, Capacitor_SMD:C_0603_1608Metric, F.Cu at (199.9, 71.0)
- added C4: 10u25v, Capacitor_SMD:C_0805_2012Metric_Pad1.15x1.40mm_HandSolder, F.Cu at (199.8, 65.7)
- added C5: 22nF, Capacitor_SMD:C_0603_1608Metric, F.Cu at (182.7, 89.1)
- added C6: 10u25v, Capacitor_SMD:C_0805_2012Metric_Pad1.15x1.40mm_HandSolder, F.Cu at (191.1, 72.3)
- added C7: 22nF, Capacitor_SMD:C_0603_1608Metric, F.Cu at (182.7, 86.6)
- added C8: 22nF, Capacitor_SMD:C_0603_1608Metric, F.Cu at (185.3, 84.1)
- added D6: BLU, LED_SMD:LED_0805_2012Metric_Pad1.15x1.40mm_HandSolder, F.Cu at (181.0, 80.5)
- added D7: 5.1V, Diode_SMD:D_SOD-123, F.Cu at (168.6, 87.2)
- added R20: 4.7k, Resistor_SMD:R_0603_1608Metric, F.Cu at (193.4, 82.1)
- added R21: 1k, Resistor_SMD:R_0603_1608Metric, F.Cu at (195.1, 76.6)
- added R22: 330, Resistor_SMD:R_0603_1608Metric, F.Cu at (199.1, 76.6)
- added R23: 1k, Resistor_SMD:R_0603_1608Metric, F.Cu at (194.1, 79.6)
- added R24: 330, Resistor_SMD:R_0603_1608Metric, F.Cu at (186.7, 86.6)
- added R25: 1k, Resistor_SMD:R_0603_1608Metric, F.Cu at (199.9, 73.5)
- added SW2: SUBCFG, kicad:TACTILE10B, F.Cu at (100.3, 102.9)
- added U7: 74LVC02APW, Package_SO:TSSOP-14_4.4x5mm_P0.65mm, F.Cu at (120.7, 142.2)
- added U8: LOADSW, Package_TO_SOT_SMD:SOT-23-6, F.Cu at (191.8, 110.5)
- added U9: LOADSW, Package_TO_SOT_SMD:SOT-23-6, F.Cu at (123.2, 120.7)
- C1, C25: value 2.2uF -> 10u25v
- C11: footprint Capacitor_SMD:C_0805_2012Metric_Pad1.15x1.40mm_HandSolder -> Capacitor_SMD:C_0603_1608Metric
- C9: value 22nF -> 10u25v
- D1: value LED -> RED
- D2: value LED -> GRN
- D4: value 3.1V Zener -> 5.1V
- J1: value USB_B_Micro -> USB
- J3: value PGDA -> UNIVERSAL; footprint Jumper:SolderJumper-3_P1.3mm_Bridged12_RoundedPad1.0x1.5mm -> Connector_PinHeader_2.54mm:PinHeader_2x07_P2.54mm_Vertical_SMD
- J8: footprint Connector_PinSocket_2.54mm:PinSocket_2x04_P2.54mm_Vertical_SMD -> Connector_PinSocket_2.54mm:PinSocket_2x05_P2.54mm_Vertical_SMD
- Q1, Q2, Q3, Q4: value 3404 -> 3402
- R1, R15, R2: footprint Resistor_SMD:R_0805_2012Metric_Pad1.15x1.40mm_HandSolder -> Resistor_SMD:R_0603_1608Metric
- R10, R12, R9: value 680 -> 100; footprint Resistor_SMD:R_0805_2012Metric_Pad1.15x1.40mm_HandSolder -> Resistor_SMD:R_0603_1608Metric
- R11, R13, R7, R8: value 220 -> 1k; footprint Resistor_SMD:R_0805_2012Metric_Pad1.15x1.40mm_HandSolder -> Resistor_SMD:R_0603_1608Metric
- R14: value 680 -> 1k; footprint Resistor_SMD:R_0805_2012Metric_Pad1.15x1.40mm_HandSolder -> Resistor_SMD:R_0603_1608Metric
- R16: value 1k -> 680
- R18: value 4.7k -> 680
- R19: value 1k -> 27k; footprint Resistor_SMD:R_0805_2012Metric_Pad1.15x1.40mm_HandSolder -> Resistor_SMD:R_0603_1608Metric
- R3: value 4.7k-1% -> 4.7k; footprint Resistor_SMD:R_0805_2012Metric_Pad1.15x1.40mm_HandSolder -> Resistor_SMD:R_0603_1608Metric
- R4, R5, R6: value 220 -> 100; footprint Resistor_SMD:R_0805_2012Metric_Pad1.15x1.40mm_HandSolder -> Resistor_SMD:R_0603_1608Metric
- U1: value STM32F042F4Px -> STM32F042; footprint Package_SO:TSSOP-20_4.4x6.5mm_P0.65mm -> Package_QFP:TQFP-32_7x7mm_P0.8mm
- U5: value EG27324 -> SP485; footprint Package_SO:SO-8_3.9x4.9mm_P1.27mm -> Package_SO:SOP-8_3.9x4.9mm_P1.27mm
- moved Q1 149.5 mm to (195.6, 101.6), turned to 0 degrees
- moved Q2 148.1 mm to (190.9, 76.0), turned to 0 degrees
- moved C23 147.8 mm to (189.2, 104.1)
- moved C9 138.2 mm to (173.9, 90.0), turned to 0 degrees
- moved L5 136.6 mm to (134.6, 132.1), turned to 180 degrees
- moved C25 123.6 mm to (88.9, 153.4), turned to 90 degrees
- moved R13 118.9 mm to (203.2, 76.0), turned to 0 degrees
- moved R12 113.4 mm to (197.4, 82.1), turned to 0 degrees
- moved R6 113.2 mm to (199.4, 68.5), turned to 0 degrees
- moved R10 112.2 mm to (194.7, 84.6)
- moved R11 109.6 mm to (190.7, 89.1)
- moved R7 107.5 mm to (190.1, 79.6)
- moved C1 101.3 mm to (173.9, 87.0)
- moved Q3 97.5 mm to (195.7, 73.1), turned to 0 degrees
- moved R5 97.1 mm to (185.4, 81.6), turned to 0 degrees
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Connections:
- C1 pad 1: PD_VDD -> VUSB
- C9 pad 1: +3V8 -> Net-(C9-Pad1)
- D1 pad 2: +3V8 -> +3V3
- D3 pad 4: WS2812 -> SPIMOSICOMB
- D4 pad 1: U2RXDIRECT -> U2RX
- J14 pad 3: WS2812 -> SPIMOSICOMB
- J3 pad 1: U2TX -> GND
- J3 pad 2: Net-(J3-Pad2) -> GND
- J3 pad 3: MAGICPIN -> VUSB
- J4 pad 2: WS2812 -> SPIMOSICOMB
- J6 pad 1: GND -> PD_VDD
- J6 pad 2: PD_VDD -> GND
- J6 pad 3: SCL -> SDA
- J6 pad 4: SDA -> SCL
- J6 pad 5: U2RX -> U2TX
- J6 pad 6: U2TX -> U2RX
- J8 pad 1: PD_VDD -> U2RX
- J8 pad 2: GND -> U2TX
- J8 pad 3: SCL -> GND
- J8 pad 4: SDA -> PD_VDD
- J8 pad 5: Net-(J3-Pad2) -> SDA
- J8 pad 6: Net-(J13-Pad2) -> SCL
- J8 pad 7: PD_VPP -> SPIMISO
- J8 pad 8: U2CK -> SPIMOSICOMB
- J9 pad 1: PD_VDD -> SPIMOSICOMB
- J9 pad 2: U2RX -> PD_VDD
- J9 pad 3: U2TX -> SPISCK
- J9 pad 4: U2CK -> SPIMISO
- J9 pad 5: GND -> MAGICPIN
- J9 pad 6: PD_VPP -> GND
- L3 pad 1: Net-(J5-Pad2) -> Net-(C23-Pad2)
- L3 pad 2: Net-(C23-Pad2) -> GND
- L4 pad 1: Net-(J7-Pad2) -> Net-(C24-Pad2)
- L4 pad 2: Net-(C24-Pad2) -> GND
- L5 pad 2: GND -> PD_VPP
- L6 pad 2: GND -> Net-(C9-Pad1)
- Q1 pad 1: TIM3_CH4 -> SW2VPP
- Q1 pad 3: Net-(C23-Pad2) -> Net-(C23-Pad1)
- Q2 pad 1: TIM16_CH1 -> SW2VDD
- Q2 pad 3: Net-(C24-Pad2) -> Net-(C24-Pad1)
- Q3 pad 1: U2RX -> DRIVELO
- Q3 pad 3: Net-(Q3-Pad3) -> MAGICPIN
- Q4 pad 1: Net-(Q4-Pad1) -> DRIVEHI
- R10 pad 1: VMON2 -> SPIMISO
- R10 pad 2: PD_VPP -> Net-(R10-Pad2)
- R11 pad 1: GND -> Net-(D6-Pad1)
- R11 pad 2: VMON2 -> SPIMISO
- R12 pad 1: VMON1 -> U2TX
- R12 pad 2: PD_VDD -> Net-(R12-Pad2)
- R13 pad 2: VMON1 -> SW1VPP
- R14 pad 2: Net-(D2-Pad1) -> SW1VPP
- R16 pad 1: MAGICPIN -> Net-(J5-Pad2)
- R16 pad 2: U2RXDIRECT -> Net-(R16-Pad2)
- R17 pad 1: Net-(C26-Pad1) -> Net-(C9-Pad1)
- R18 pad 1: MAGICPIN -> Net-(J7-Pad2)
- R18 pad 2: MPMON -> Net-(R18-Pad2)
- R19 pad 1: MPMON -> PD_VPP
- R19 pad 2: GND -> Net-(Q5-Pad1)
- R3 pad 2: TIM16_CH1 -> Net-(R3-Pad2)
- R5 pad 1: SCL -> Net-(R5-Pad1)
- R5 pad 2: Net-(R5-Pad2) -> SPIMOSICOMB
- R6 pad 1: U2CK -> SCL
- R7 pad 1: U2TX -> Net-(D1-Pad1)
- R7 pad 2: SWC -> U2RX
- R8 pad 1: U2RX -> Net-(D2-Pad1)
- R8 pad 2: U2RXDIRECT -> GND
- R9 pad 1: Net-(Q3-Pad3) -> U2CK
- R9 pad 2: Net-(D1-Pad1) -> Net-(R9-Pad2)
- SW1 pad 4: TIM16_CH1 -> Net-(R3-Pad2)
- U1 pad 1: TIM16_CH1 -> +3V3
- U1 pad 10: Net-(R6-Pad2) -> Net-(R9-Pad2)
- U1 pad 12: MPMON -> Net-(R10-Pad2)
- U1 pad 13: WS2812 -> PIMON
- U1 pad 14: TIM3_CH4 -> SW1VDD
- U1 pad 15: GND -> SW2VDD
- U1 pad 16: +3V3 -> GND
- U1 pad 17: D- -> +3V3
- U1 pad 18: D+ -> SW1VPP
- U1 pad 19: SWD -> SW2VPP
- U1 pad 20: SWC -> Net-(U1-Pad20)
- U1 pad 3: Net-(R5-Pad2) -> Net-(R6-Pad2)
- U1 pad 8: PIMON -> Net-(R12-Pad2)
- U1 pad 9: U2RXDIRECT -> Net-(R12-Pad2)
- U5 pad 1: Net-(U5-Pad1) -> U2RX
- U5 pad 2: U2TX -> ~485RXEN~
- U5 pad 3: GND -> U2TXEN
- U5 pad 5: Net-(Q6-Pad1) -> GND
- U5 pad 6: PD_VPP -> 485A
- U5 pad 7: Net-(Q4-Pad1) -> 485B
- U5 pad 8: U2RTS -> VUSB
- U6 pad 3: Net-(C26-Pad1) -> Net-(C9-Pad1)
Other:
- board text added: "1.65mm Component Thickness (TQFP 1.6 + SOIC-8 1.7 + LED 1.5)"
- board text added: "GND GND +5V VDD UTX SCK SWD URX 458- RTS 485+ VPP GND MP"
- board text added: "UTX URX VDD GND SCL SDA IPD PA4 VPP IPC"
- board text removed: "GND VDD SDA SCL DX DAT CLK PGM"
- board text removed: "NPX VPP SCL SDA UCK VDD DRX MAG DTX GND"
- board text removed: "VDD ARX ATX UCK GND VPP"

Commit message: Progress on multitool
Parts:
- removed L2: 10uH, Inductor_SMD:L_2816_7142Metric
- added C10: 22nF, Capacitor_SMD:C_0603_1608Metric, F.Cu at (101.2, 118.5)
- added C12: 22nF, Capacitor_SMD:C_0603_1608Metric, F.Cu at (97.9, 145.5)
- added D8: 5.1V, Diode_SMD:D_SOD-123, F.Cu at (136.1, 153.1)
- added R26: 4.7k, Resistor_SMD:R_0603_1608Metric, F.Cu at (143.6, 162.1)
- added R27: 4.7k, Resistor_SMD:R_0603_1608Metric, F.Cu at (139.8, 162.1)
- added U10: 3v6, Package_TO_SOT_SMD:SOT-23, F.Cu at (102.4, 127.2)
- C6: value 10u25v -> 10u
- Q5: value Q_PNP_BEC -> PNP
- R16, R18: value 680 -> 330; footprint Resistor_SMD:R_0805_2012Metric_Pad1.15x1.40mm_HandSolder -> Resistor_SMD:R_0603_1608Metric
- U4: value XC6206P360MR -> 3v6
- moved D6 138.5 mm to (94.8, 189.0), turned to 270 degrees
- moved R7 136.5 mm to (104.2, 185.6), turned to 90 degrees
- moved R11 136.0 mm to (94.8, 185.5), turned to 90 degrees
- moved C3 125.4 mm to (86.5, 124.6)
- moved R6 122.9 mm to (97.5, 137.1), turned to 90 degrees
- moved R8 117.3 mm to (99.4, 185.5), turned to 90 degrees
- moved D7 113.2 mm to (93.6, 172.0), turned to 90 degrees
- moved R10 111.8 mm to (94.8, 134.9), turned to 60 degrees
- moved L4 110.9 mm to (143.4, 122.4), turned to 180 degrees
- moved R25 106.5 mm to (129.8, 153.6), turned to 270 degrees
- moved Q3 103.8 mm to (119.9, 144.1)
- moved C6 102.9 mm to (104.8, 128.5), turned to 240 degrees
- moved J7 101.8 mm to (139.6, 111.9), turned to 300 degrees
- moved R5 97.3 mm to (112.6, 146.3), turned to 270 degrees
- moved R21 96.1 mm to (124.3, 141.5), turned to 180 degrees
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Connections:
- D3 pad 6: GND -> PA10
- J3 pad 10: U2RTS -> Net-(J3-Pad10)
- J3 pad 14: MAGICPIN -> U2CK
- R14 pad 2: SW1VPP -> SW1VDD
- R23 pad 1: Net-(C9-Pad1) -> PD_VDD
- R5 pad 1: Net-(R5-Pad1) -> U2RTS
- R5 pad 2: SPIMOSICOMB -> Net-(J3-Pad10)
- U1 pad 20: Net-(U1-Pad20) -> PA10
- U1 pad 27: Net-(R5-Pad1) -> SPIMOSICOMB
- U1 pad 28: Net-(R5-Pad1) -> SPIMOSICOMB
Routing:
- net GND: track 0.00 -> 186.2 mm, vias 0 -> 9
- net VUSB: track 0.00 -> 176.7 mm, vias 0 -> 7
- net SPISCK: track 0.00 -> 128.3 mm, vias 0 -> 2
- net U2RX: track 0.00 -> 123.9 mm, vias 0 -> 5
- net SPIMOSICOMB: track 0.00 -> 83.6 mm, vias 0 -> 2
- net +3V8: track 0.00 -> 73.4 mm, vias 0 -> 7
- net SPIMISO: track 0.00 -> 71.2 mm, vias 0 -> 2
- net U2TX: track 0.00 -> 67.2 mm, vias 0 -> 3
- net PD_VDD: track 0.00 -> 61.7 mm, vias 0 -> 3
- net Net-(R3-Pad2): track 0.00 -> 55.7 mm, vias 0 -> 2
- net SWD: track 0.00 -> 45.5 mm
- net SWC: track 0.00 -> 43.4 mm
- net MAGICPIN: track 0.00 -> 39.2 mm, vias 0 -> 2
- net ~485RXEN~: track 0.00 -> 32.7 mm, vias 0 -> 2
- net NRST: track 0.00 -> 32.0 mm
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Other:
- net class Default: clearance 0.199 -> 0.2159; trace_width 0.3 -> 0.3048
- rule trace_clearance: 0.199 -> 0.2159

Commit message: bump design slightly.
Parts:
- removed D3: WS2813, LED_SMD:LED_WS2812_PLCC6_5.0x5.0mm_P1.6mm
- removed J14: WS2813, Connector_PinHeader_2.54mm:PinHeader_1x04_P2.54mm_Vertical_SMD_Pin1Right
- added J10: SMARTLED, Connector_PinHeader_2.54mm:PinHeader_1x04_P2.54mm_Vertical_SMD_Pin1Left, F.Cu at (142.2, 171.3)
- added U11: 74AHCT1G126, Package_TO_SOT_SMD:SOT-23-6, F.Cu at (130.4, 154.4)
- added U12: 74AHCT1G126, Package_TO_SOT_SMD:SOT-23-6, F.Cu at (130.4, 161.8)
- J1: footprint kicad:USBMicroB-U253-051T-4BH89-F1B -> chinese-connectors:chinausb-multi
- R11, R25, R7, R8: value 1k -> 4.7k
- moved J16 76.6 mm to (99.0, 111.9), turned to 90 degrees
- moved R25 7.87 mm to (125.9, 160.4), turned to 90 degrees
- moved R7 7.78 mm to (96.4, 184.8), turned to 270 degrees
- moved R11 7.52 mm to (102.3, 184.7), turned to 270 degrees
- moved D1 2.49 mm to (101.7, 189.0)
- moved D6 2.26 mm to (97.1, 189.0)
- moved R8 0.78 mm to (99.4, 184.7), turned to 270 degrees
- moved J1 0.72 mm to (114.3, 98.5), turned to 0 degrees
- moved U3 0.66 mm to (114.7, 105.0)
Connections:
- J4 pad 2: SPIMOSICOMB -> Net-(J10-Pad3)
- R11 pad 1: Net-(D6-Pad1) -> SPIMISO
- R11 pad 2: SPIMISO -> Net-(D1-Pad1)
- R25 pad 1: MAGICPIN -> U2RX
- R25 pad 2: U2RX -> MAGICPIN
- R7 pad 1: Net-(D1-Pad1) -> U2RX
- R7 pad 2: U2RX -> Net-(D6-Pad1)
- R8 pad 1: Net-(D2-Pad1) -> GND
- R8 pad 2: GND -> Net-(D2-Pad1)
Routing:
- net GND: track 186.2 -> 215.3 mm, vias 9 -> 11
- net VUSB: track 176.7 -> 156.3 mm
- net U2RX: track 123.9 -> 142.4 mm
- net +3V8: track 73.4 -> 89.8 mm, vias 7 -> 8
- net +3V3: track 31.0 -> 19.2 mm
- net SPIMISO: track 71.2 -> 77.5 mm
- net D-: track 13.8 -> 10.4 mm
- net D+: track 12.9 -> 11.1 mm
- net SPIMOSICOMB: track 83.6 -> 85.2 mm
- net PD_VDD: track 61.7 -> 60.4 mm, vias 3 -> 5
- net Net-(D1-Pad1): track 1.66 -> 2.54 mm
- net Net-(D2-Pad1): track 1.66 -> 2.45 mm
- net Net-(D6-Pad1): track 1.71 -> 2.48 mm

Commit message: bump
Parts:
- moved R26 47.6 mm to (118.2, 121.9), turned to 90 degrees
- moved R27 29.0 mm to (128.7, 189.0), turned to 180 degrees
- moved U12 23.5 mm to (129.8, 185.2)
- moved R25 14.8 mm to (115.7, 149.8), turned to 0 degrees
- moved R16 4.39 mm to (124.1, 122.3), turned to 180 degrees
- moved L4 1.73 mm to (141.7, 122.5)
- moved C19 1.16 mm to (116.8, 112.6)
- moved C24 1.05 mm to (145.2, 127.3)
- moved L6 0.67 mm to (144.3, 134.1)
- moved R6 0.37 mm to (97.6, 137.5)
- moved C9 0.35 mm to (139.4, 134.4)
- moved J1 0.08 mm to (114.3, 98.6)
Routing:
- net GND: track 215.3 -> 1159.0 mm, vias 11 -> 124
- net +3V3: track 19.2 -> 156.8 mm, vias 0 -> 5
- net VUSB: track 156.3 -> 286.5 mm, vias 7 -> 11
- net PD_VDD: track 60.4 -> 167.6 mm, vias 5 -> 10
- net U2CK: track 0.00 -> 93.1 mm, vias 0 -> 4
- net SWD: track 45.5 -> 136.4 mm, vias 0 -> 2
- net U2TX: track 67.2 -> 154.0 mm, vias 3 -> 10
- net PD_VPP: track 0.00 -> 70.2 mm, vias 0 -> 5
- net SCL: track 27.2 -> 97.0 mm, vias 0 -> 3
- net 485A: track 0.00 -> 59.6 mm, vias 0 -> 2
- net 485B: track 0.00 -> 59.3 mm, vias 0 -> 2
- net U2RX: track 142.4 -> 201.6 mm, vias 5 -> 10
- net SPIMOSICOMB: track 85.2 -> 136.3 mm, vias 2 -> 4
- net MAGICPIN: track 39.2 -> 89.8 mm, vias 2 -> 5
- net SDA: track 24.2 -> 73.4 mm
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- added copper zone on B.Cu, net GND
- added copper zone on F.Cu, net GND

Commit message: bump design
Parts:
- moved C2 0.57 mm to (132.1, 114.7)
Routing:
- net GND: track 1159.0 -> 1185.7 mm, vias 124 -> 126

Commit message: bump
Other:
- board text added: "TX GND EN G2 RST G0 5V RX"
