File: stm32f042_breakout/stm32f042_breakout.sch (KiCad schematic (older format))
At the start: 32 parts, among them J1 PGM, J10 MNT, J11 MNT, J12 MNT, J13 MNT, J2 USB_B_Micro, J3 PORTB, J4 PORTB, J5 POWER, J6 3.3v REG SW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

Commit message: Add the breakout, as printed.
Parts:
- added J14: ARTWORK, stm32f042_breakout:back-artwork-cristabelle-braden-vsmall, symbol Connector_Generic:Conn_01x01
- added J15: ARTWORK, stm32f042_breakout:leaves_front-cristabelle, symbol Connector_Generic:Conn_01x01
- added J16: ARTWORK, stm32f042_breakout:cb-signature, symbol Connector_Generic:Conn_01x01
- added JP1: EN_XTAL, Jumper:SolderJumper-2_P1.3mm_Bridged_RoundedPad1.0x1.5mm, symbol Jumper:SolderJumper_2_Bridged
- C3, C4, C8, C9: value 100n -> .1u
- J10, J11, J12, J13, J8, J9: footprint MountingHole:MountingHole_4.3mm_M4_DIN965 -> stm32f042_breakout:stm32f042_breakout_pin
- J4: value PORTB -> PORTA
Connections:
- net at C5.2, C6.2, Y1.1: now also JP1.1 (A); no longer U3.2 (PF0)
- new net: JP1.2 (B), U3.2 (PF0)
Changed lines of the file:
@@
 P 1100 900
 F 0 "C4" H 1050 1000 50  0000 R CNN
-F 1 "100n" H 1300 800 50  0000 R CNN
+F 1 ".1u" H 1300 800 50  0000 R CNN
 F 2 "Capacitor_SMD:C_0603_1608Metric" H 1100 900 50  0001 C CNN
 F 3 "~" H 1100 900 50  0001 C CNN
@@
 P 1050 3400
 F 0 "C3" H 1000 3500 50  0000 R CNN
-F 1 "100n" H 1250 3300 50  0000 R CNN
+F 1 ".1u" H 1250 3300 50  0000 R CNN
 F 2 "Capacitor_SMD:C_0603_1608Metric" H 1050 3400 50  0001 C CNN
 F 3 "~" H 1050 3400 50  0001 C CNN
@@
 P 8350 3300
 F 0 "C8" H 8300 3400 50  0000 R CNN
-F 1 "100n" H 8550 3200 50  0000 R CNN
+F 1 ".1u" H 8550 3200 50  0000 R CNN
 F 2 "Capacitor_SMD:C_0603_1608Metric" H 8350 3300 50  0001 C CNN
 F 3 "~" H 8350 3300 50  0001 C CNN
@@
 BOOT0
 Wire Wire Line
-	2200 1700 2650 1700
-Connection ~ 2200 1700
-Wire Wire Line
 	1850 1700 1850 1600
 Connection ~ 1850 1700
@@
 	2200 1600 2200 1700
 Wire Wire Line
-	1850 1600 2200 1600
+	1850 1600 2000 1600
 Wire Wire Line
 	1850 1800 1850 1700
@@
 P 5100 2900
 F 0 "J4" H 5150 3517 50  0000 C CNN
-F 1 "PORTB" H 5150 3426 50  0000 C CNN
+F 1 "PORTA" H 5150 3426 50  0000 C CNN
 F 2 "Connector_PinHeader_2.54mm:PinHeader_2x09_P2.54mm_Vertical_SMD" H 5100 2900 50  0001 C CNN
 F 3 "~" H 5100 2900 50  0001 C CNN
@@
 P 3900 850
 F 0 "C9" H 3850 950 50  0000 R CNN
-F 1 "100n" H 4100 750 50  0000 R CNN
+F 1 ".1u" H 4100 750 50  0000 R CNN
 F 2 "Capacitor_SMD:C_0603_1608Metric" H 3900 850 50  0001 C CNN
 F 3 "~" H 3900 850 50  0001 C CNN
@@
 F 0 "J13" H 6268 4175 50  0000 C CNN
 F 1 "MNT" H 6268 4266 50  0000 C CNN
-F 2 "MountingHole:MountingHole_4.3mm_M4_DIN965" H 6350 4400 50  0001 C CNN
+F 2 "stm32f042_breakout:stm32f042_breakout_pin" H 6350 4400 50  0001 C CNN
 F 3 "~" H 6350 4400 50  0001 C CNN
 	1    6350 4400
@@
 F 0 "J10" H 5668 3675 50  0000 C CNN
 F 1 "MNT" H 5668 3766 50  0000 C CNN
-F 2 "MountingHole:MountingHole_4.3mm_M4_DIN965" H 5750 3900 50  0001 C CNN
+F 2 "stm32f042_breakout:stm32f042_breakout_pin" H 5750 3900 50  0001 C CNN
 F 3 "~" H 5750 3900 50  0001 C CNN
 	1    5750 3900
@@
 F 0 "J11" H 5668 3975 50  0000 C CNN
 F 1 "MNT" H 5668 4066 50  0000 C CNN
-F 2 "MountingHole:MountingHole_4.3mm_M4_DIN965" H 5750 4200 50  0001 C CNN
+F 2 "stm32f042_breakout:stm32f042_breakout_pin" H 5750 4200 50  0001 C CNN
 F 3 "~" H 5750 4200 50  0001 C CNN
 	1    5750 4200
@@
 F 0 "J12" H 5668 4325 50  0000 C CNN
 F 1 "MNT" H 5668 4416 50  0000 C CNN
-F 2 "MountingHole:MountingHole_4.3mm_M4_DIN965" H 5750 4550 50  0001 C CNN
+F 2 "stm32f042_breakout:stm32f042_breakout_pin" H 5750 4550 50  0001 C CNN
 F 3 "~" H 5750 4550 50  0001 C CNN
 	1    5750 4550
@@
 F 0 "J9" H 5168 4175 50  0000 C CNN
 F 1 "MNT" H 5168 4266 50  0000 C CNN
-F 2 "MountingHole:MountingHole_4.3mm_M4_DIN965" H 5250 4400 50  0001 C CNN
+F 2 "stm32f042_breakout:stm32f042_breakout_pin" H 5250 4400 50  0001 C CNN
 F 3 "~" H 5250 4400 50  0001 C CNN
 	1    5250 4400
@@
 F 0 "J8" H 5168 3775 50  0000 C CNN
 F 1 "MNT" H 5168 3866 50  0000 C CNN
-F 2 "MountingHole:MountingHole_4.3mm_M4_DIN965" H 5250 4000 50  0001 C CNN
+F 2 "stm32f042_breakout:stm32f042_breakout_pin" H 5250 4000 50  0001 C CNN
 F 3 "~" H 5250 4000 50  0001 C CNN
 	1    5250 4000
 	-1   0    0    1
 $EndComp
+$Comp
+L Connector_Generic:Conn_01x01 J14
+U 1 1 5F1B7109
+P 7250 4500
+F 0 "J14" H 7168 4275 50  0000 C CNN
+F 1 "ARTWORK" H 7168 4366 50  0000 C CNN
+F 2 "stm32f042_breakout:back-artwork-cristabelle-braden-vsmall" H 7250 4500 50  0001 C CNN
+F 3 "~" H 7250 4500 50  0001 C CNN
+	1    7250 4500
+	-1   0    0    1
+$EndComp
+$Comp
+L Jumper:SolderJumper_2_Bridged JP1
+U 1 1 5F1D47AC
+P 2150 1400
+F 0 "JP1" H 2150 1605 50  0000 C CNN
+F 1 "EN_XTAL" H 2150 1514 50  0000 C CNN
+F 2 "Jumper:SolderJumper-2_P1.3mm_Bridged_RoundedPad1.0x1.5mm" H 2150 1400 50  0001 C CNN
+F 3 "~" H 2150 1400 50  0001 C CNN
+	1    2150 1400
+	1    0    0    -1
+$EndComp
+Wire Wire Line
+	2000 1400 2000 1600
+Connection ~ 2000 1600
+Wire Wire Line
+	2000 1600 2200 1600
+Wire Wire Line
+	2300 1400 2300 1700
+Wire Wire Line
+	2300 1700 2650 1700
+$Comp
+L Connector_Generic:Conn_01x01 J15
+U 1 1 5F1B9EC9
+P 7700 4500
+F 0 "J15" H 7618 4275 50  0000 C CNN
+F 1 "ARTWORK" H 7618 4366 50  0000 C CNN
+F 2 "stm32f042_breakout:leaves_front-cristabelle" H 7700 4500 50  0001 C CNN
+F 3 "~" H 7700 4500 50  0001 C CNN
+	1    7700 4500
+	-1   0    0    1
+$EndComp
+$Comp
+L Connector_Generic:Conn_01x01 J16
+U 1 1 5F1E7A36
+P 8200 4500
+F 0 "J16" H 8118 4275 50  0000 C CNN
+F 1 "ARTWORK" H 8118 4366 50  0000 C CNN
+F 2 "stm32f042_breakout:cb-signature" H 8200 4500 50  0001 C CNN
+F 3 "~" H 8200 4500 50  0001 C CNN
+	1    8200 4500
+	-1   0    0    1
+$EndComp
