File: multitool-attempt-at-can/multitool.sch (KiCad schematic (older format))
At the start: 90 parts, among them J1 USB, J14 WS2813, J15 ESP-01, J16 VDDS, J17 MNT, J18 MNT, J19 MNT, J2 SELF_PGM, J20 MNT, J3 UNIVERSAL, J4 WSOUT, J5 VPPS, J6 SAO, J7 VDDS, J8 PADAUK, J9 AVR, Q1 3402, Q2 3402, Q3 3402, Q4 3402, Q5 PNP, SW1 BOOT0, SW2 SUBCFG, U1 STM32F042, U10 3v6, U2 MT2492, U3 NUP4202, U4 3v6, U5 SP485, U6 INA181A3, U7 74LVC02APW, U8 LOADSW, U9 LOADSW

Commit message: Move attempt at can away.
Parts:
- removed U1: STM32F042, Package_QFP:TQFP-32_7x7mm_P0.8mm, symbol MCU_ST_STM32F0:STM32F042K4Tx
- added U?: STM32F042C6Tx, Package_QFP:LQFP-48_7x7mm_P0.5mm, symbol MCU_ST_STM32F0:STM32F042C6Tx
- gave numbers to parts that had none: 1
Connections:
- net labels added: BOOT0, CANRX, CANTX, SUBCFG, U2TXRX, VMONIN
- net labels removed: U2TX
- wire segments 111 -> 98
Other:
- note added: "Inductors: https://lcsc.com/product-detail/Power-Inductors_Ceaiya-CR5040-220M_C520354.html (22uH)\nor \nhttps://lcsc.com/product-detail/New-Quadratic-Unclassified-Data_GLE-GCNR4030-100MC_C439346.html (10uH)"
- note added: "T16C1"
- note added: "T2C3\nT2C4"
- note added: "TODO: REDO GPIO"
- note added: "U2RX is 5V tolerant\nSPISCK is 5V tolerant"
- note removed: "T1C1\nT1C2"
- note removed: "T2CH3"
- note removed: "U2TX alt is TIM2_CH3"
- note removed: "U2TX can also function as SPI_NSS\nU2RX is 5V tolerant\nSPISCK is 5V tolerant"
- moved on the sheet: C10, C19, C23, C25, C6, C7, C8, D23, J2, J5, J7, L3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
